Commit message: Modified Universal Robot launch

File: cooperative_manipulation_robot_description/custom_ur_description/ur16e_urdf/custom_ur16e_robot.urdf.xacro (robot description, xacro)
@@ -2,4 +2,6 @@
 <robot xmlns:xacro="http://ros.org/wiki/xacro"
        name="ur16e" >
+  <xacro:arg name="xyz" default="'0 0 0'"/>
+  <xacro:arg name="rpy" default="'0 0 0'"/>
   <!-- common stuff -->
   <xacro:include filename="$(find ur_e_description)/urdf/common.gazebo.xacro" />
@@ -15,5 +17,5 @@
     <parent link="world" />
     <child link = "base_link" />
-    <origin xyz="0.0 0.0 0.0" rpy="0.0 0.0 0.0" />
+    <origin xyz="$(arg xyz)" rpy="$(arg rpy)" />
   </joint>
 </robot>
