Commit message: Modified Universal Robot .laund and urdf

File: cooperative_manipulation_robot_description/custom_ur_description/ur16e_urdf/custom_ur16e_joint_limited_robot.urdf.xacro (robot description, xacro)
@@ -1,7 +1,6 @@
 <?xml version="1.0"?>
 <robot xmlns:xacro="http://ros.org/wiki/xacro"
-       name="ur16e" >
-  <xacro:arg name="xyz" default="'0 0 0'"/>
-  <xacro:arg name="rpy" default="'0 0 0'"/>
+  name="ur16e" >
+  <xacro:arg name="transmission_hw_interface" default="hardware_interface/VelocityJointInterface"/>
   <!-- common stuff -->
   <xacro:include filename="$(find cooperative_manipulation_robot_description)/custom_ur_description/ur16e_urdf/custom_common.gazebo.xacro" />
@@ -10,12 +9,19 @@
   <!-- arm -->
   <xacro:arg name="kinematics_config" default="$(find ur_e_description)/config/ur16e_default.yaml"/>
-  <xacro:ur16e_robot prefix="" joint_limited="false"
+  <xacro:ur16e_robot prefix="" joint_limited="true"
+    shoulder_pan_lower_limit="${-pi}" shoulder_pan_upper_limit="${pi}"
+    shoulder_lift_lower_limit="${-pi}" shoulder_lift_upper_limit="${pi}"
+    elbow_joint_lower_limit="${-pi}" elbow_joint_upper_limit="${pi}"
+    wrist_1_lower_limit="${-pi}" wrist_1_upper_limit="${pi}"
+    wrist_2_lower_limit="${-pi}" wrist_2_upper_limit="${pi}"
+    wrist_3_lower_limit="${-pi}" wrist_3_upper_limit="${pi}"
+    transmission_hw_interface="$(arg transmission_hw_interface)"
     kinematics_file="${load_yaml('$(arg kinematics_config)')}"
-  />
+    />
   <link name="world" />
   <joint name="world_joint" type="fixed">
     <parent link="world" />
     <child link = "base_link" />
-    <origin xyz="$(arg xyz)" rpy="$(arg rpy)" />
+    <origin xyz="0.0 0.0 0.0" rpy="0.0 0.0 0.0" />
   </joint>
 </robot>

Commit message: Modified launch files to set correct pose for both robots

File: cooperative_manipulation_robot_description/custom_ur_description/ur16e_urdf/custom_ur16e_joint_limited_robot.urdf.xacro (robot description, xacro)
@@ -2,4 +2,6 @@
 <robot xmlns:xacro="http://ros.org/wiki/xacro"
   name="ur16e" >
+  <xacro:arg name="xyz" default="'0 0 0'"/>
+  <xacro:arg name="rpy" default="'0 0 0'"/>
   <xacro:arg name="transmission_hw_interface" default="hardware_interface/VelocityJointInterface"/>
   <!-- common stuff -->
@@ -23,5 +25,5 @@
     <parent link="world" />
     <child link = "base_link" />
-    <origin xyz="0.0 0.0 0.0" rpy="0.0 0.0 0.0" />
+    <origin xyz="$(arg xyz)" rpy="$(arg rpy)" />
   </joint>
 </robot>

File: cooperative_manipulation_robot_description/custom_ur_description/ur16e_urdf/custom_ur16e_robot.urdf.xacro (robot description, xacro)
@@ -9,5 +9,5 @@
   <xacro:include filename="$(find cooperative_manipulation_robot_description)/custom_ur_description/ur16e_urdf/custom_ur16e.urdf.xacro" />
   <!-- arm -->
-  <xacro:arg name="kinematics_config" default="$(find ur_e_description)/config/ur16e_default.yaml"/>
+  <xacro:arg name="kinematics_config" default="$(find cooperative_manipulation_robot_description)/custom_ur_description/config/custom_ur16e_default.yaml"/>
   <xacro:ur16e_robot prefix="" joint_limited="false"
     kinematics_file="${load_yaml('$(arg kinematics_config)')}"
